File: hw/sch_pcb/Connectors.kicad_sch (KiCad schematic)
At the start: 6 parts, among them J10 HEADER_2x05_PARALLEL, J11 HEADER_2x07_PARALLEL, J12 HEADER_2x05_PARALLEL, J7 Conn_01x06_Female, J8 Conn_01x07_Female, J9 Conn_01x04_Female

Commit message: Update project to KiCADv9.
Other:
- title: (none) -> DATALOGGER02A
Changed lines of the file:
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@@
 (kicad_sch
-	(version 20231120)
+	(version 20250114)
 	(generator "eeschema")
-	(generator_version "8.0")
+	(generator_version "9.0")
 	(paper "A4")
+	(title_block
+		(title "DATALOGGER02A")
+	)
+	(text "3V3"
+		(exclude_from_sim no)
+		(at 83.82 113.03 0)
+		(effects
+			(font
+				(size 1.524 1.524)
+			)
+			(justify left bottom)
+		)
+	)
+	(text "3V3"
+		(exclude_from_sim no)
+		(at 83.82 120.65 0)
+		(effects
+			(font
+				(size 1.524 1.524)
+			)
+			(justify left bottom)
+		)
+	)
+	(text "3V3"
+		(exclude_from_sim no)
+		(at 81.28 77.47 0)
+		(effects
+			(font
+				(size 1.524 1.524)
+			)
+			(justify left bottom)
+		)
+	)
+	(text "ANALOG CONN"
+		(exclude_from_sim no)
+		(at 169.672 62.23 0)
+		(effects
+			(font
+				(size 3 3)
+			)
+			(justify left bottom)
+		)
+	)
+	(text "3V3"
+		(exclude_from_sim no)
+		(at 83.82 118.11 0)
+		(effects
+			(font
+				(size 1.524 1.524)
+			)
+			(justify left bottom)
+		)
+	)
+	(text "I2C CONN"
+		(exclude_from_sim no)
+		(at 173.99 100.33 0)
+		(effects
+			(font
+				(size 3 3)
+			)
+			(justify left bottom)
+		)
+	)
+	(text "3V3"
+		(exclude_from_sim no)
+		(at 127 76.2 0)
+		(effects
+			(font
+				(size 1.524 1.524)
+			)
+			(justify left bottom)
+		)
+	)
+	(text "I2C CONN."
+		(exclude_from_sim no)
+		(at 118.11 64.77 0)
+		(effects
+			(font
+				(size 3 3)
+			)
+			(justify left bottom)
+		)
+	)
+	(text "3V3"
+		(exclude_from_sim no)
+		(at 83.82 115.57 0)
+		(effects
+			(font
+				(size 1.524 1.524)
+			)
+			(justify left bottom)
+		)
+	)
+	(text "AUX_I2C CONN"
+		(exclude_from_sim no)
+		(at 209.55 64.77 0)
+		(effects
+			(font
+				(size 3 3)
+			)
+			(justify left bottom)
+		)
+	)
+	(text "3V3"
+		(exclude_from_sim no)
+		(at 83.82 110.49 0)
+		(effects
+			(font
+				(size 1.524 1.524)
+			)
+			(justify left bottom)
+		)
+	)
+	(text "3V3"
+		(exclude_from_sim no)
+		(at 81.28 80.01 0)
+		(effects
+			(font
+				(size 1.524 1.524)
+			)
+			(justify left bottom)
+		)
+	)
+	(text "PIN HEADERS"
+		(exclude_from_sim no)
+		(at 163.83 55.88 0)
+		(effects
+			(font
+				(size 3 3)
+			)
+			(justify left bottom)
+		)
+	)
+	(text "SPI CONN."
+		(exclude_from_sim no)
+		(at 74.93 99.06 0)
+		(effects
+			(font
+				(size 3 3)
+			)
+			(justify left bottom)
+		)
+	)
+	(text "3V3"
+		(exclude_from_sim no)
+		(at 127 78.74 0)
+		(effects
+			(font
+				(size 1.524 1.524)
+			)
+			(justify left bottom)
+		)
+	)
+	(text "UART CONN."
+		(exclude_from_sim no)
+		(at 72.39 64.77 0)
+		(effects
+			(font
+				(size 3 3)
+			)
+			(justify left bottom)
+		)
+	)
+	(text "PIXHAWK STANDARD HEADERS"
+		(exclude_from_sim no)
+		(at 67.31 55.88 0)
+		(effects
+			(font
+				(size 3 3)
+			)
+			(justify left bottom)
+		)
+	)
 	(junction
 		(at 223.52 77.47)
@@
 		)
 	)
-	(text "3V3"
-		(exclude_from_sim no)
-		(at 83.82 113.03 0)
-		(effects
-			(font
-				(size 1.524 1.524)
-			)
-			(justify left bottom)
-		)
-	)
-	(text "3V3"
-		(exclude_from_sim no)
-		(at 83.82 120.65 0)
-		(effects
-			(font
-				(size 1.524 1.524)
-			)
-			(justify left bottom)
-		)
-	)
-	(text "3V3"
-		(exclude_from_sim no)
-		(at 81.28 77.47 0)
-		(effects
-			(font
-				(size 1.524 1.524)
-			)
-			(justify left bottom)
-		)
-	)
-	(text "ANALOG CONN"
-		(exclude_from_sim no)
-		(at 169.672 62.23 0)
-		(effects
-			(font
-				(size 3 3)
-			)
-			(justify left bottom)
-		)
-	)
-	(text "3V3"
-		(exclude_from_sim no)
-		(at 83.82 118.11 0)
-		(effects
-			(font
-				(size 1.524 1.524)
-			)
-			(justify left bottom)
-		)
-	)
-	(text "I2C CONN"
-		(exclude_from_sim no)
-		(at 173.99 100.33 0)
-		(effects
-			(font
-				(size 3 3)
-			)
-			(justify left bottom)
-		)
-	)
-	(text "3V3"
-		(exclude_from_sim no)
-		(at 127 76.2 0)
-		(effects
-			(font
-				(size 1.524 1.524)
-			)
-			(justify left bottom)
-		)
-	)
-	(text "I2C CONN."
-		(exclude_from_sim no)
-		(at 118.11 64.77 0)
-		(effects
-			(font
-				(size 3 3)
-			)
-			(justify left bottom)
-		)
-	)
-	(text "3V3"
-		(exclude_from_sim no)
-		(at 83.82 115.57 0)
-		(effects
-			(font
-				(size 1.524 1.524)
-			)
-			(justify left bottom)
-		)
-	)
-	(text "AUX_I2C CONN"
-		(exclude_from_sim no)
-		(at 209.55 64.77 0)
-		(effects
-			(font
-				(size 3 3)
-			)
-			(justify left bottom)
-		)
-	)
-	(text "3V3"
-		(exclude_from_sim no)
-		(at 83.82 110.49 0)
-		(effects
-			(font
-				(size 1.524 1.524)
-			)
-			(justify left bottom)
-		)
-	)
-	(text "3V3"
-		(exclude_from_sim no)
-		(at 81.28 80.01 0)
-		(effects
-			(font
-				(size 1.524 1.524)
-			)
-			(justify left bottom)
-		)
-	)
-	(text "PIN HEADERS"
-		(exclude_from_sim no)
-		(at 163.83 55.88 0)
-		(effects
-			(font
-				(size 3 3)
-			)
-			(justify left bottom)
-		)
-	)
-	(text "SPI CONN."
-		(exclude_from_sim no)
-		(at 74.93 99.06 0)
-		(effects
-			(font
-				(size 3 3)
-			)
-			(justify left bottom)
-		)
-	)
-	(text "3V3"
-		(exclude_from_sim no)
-		(at 127 78.74 0)
-		(effects
-			(font
-				(size 1.524 1.524)
-			)
-			(justify left bottom)
-		)
-	)
-	(text "UART CONN."
-		(exclude_from_sim no)
-		(at 72.39 64.77 0)
-		(effects
-			(font
-				(size 3 3)
-			)
-			(justify left bottom)
-		)
-	)
-	(text "PIXHAWK STANDARD HEADERS"
-		(exclude_from_sim no)
-		(at 67.31 55.88 0)
-		(effects
-			(font
-				(size 3 3)
-			)
-			(justify left bottom)
-		)
-	)
