File: hw/sch_pcb/Connectors.kicad_sch (KiCad schematic)
At the start: 6 parts, among them J10 HEADER_2x05_PARALLEL, J11 HEADER_2x07_PARALLEL, J12 HEADER_2x05_PARALLEL, J7 Conn_01x06_Female, J8 Conn_01x07_Female, J9 Conn_01x04_Female

Commit message: Desing improvements WIP.
Parts:
- added J14: Conn_01x06_Female, Connector_JST:JST_GH_SM06B-GHS-TB_1x06-1MP_P1.25mm_Horizontal, symbol Connector:Conn_01x06_Female
Connections:
- net +5V: now also J14.1 (Pin_1)
- net GND: now also J14.6 (Pin_6)
- net RX1: now also J14.3 (Pin_3)
- net TX1: now also J14.2 (Pin_2)
- no-connect marks 2 -> 4
Other:
- note added: "I2C"
- note added: "MLAB Pin Headers"
- note added: "Pixhawk connectors"
- note added: "SPI"
- note added: "UART (FMU)"
- note added: "UART (Peripheral)"
- note removed: "I2C CONN"
- note removed: "I2C CONN."
- note removed: "PIN HEADERS"
- note removed: "PIXHAWK STANDARD HEADERS"
- note removed: "SPI CONN."
- note removed: "UART CONN."
- moved on the sheet: J7, J8, J9
