File: hw/sch_pcb/Microcontroller.kicad_sch (KiCad schematic)
At the start: 28 parts, among them J1 HEADER_2x01_PARALLEL, J2 HEADER_2x01, J3 HEADER_2x03, U1 ISL21080CIH320Z-TK, U2 LM4041CIM3-1.2(neosazovat), U3 ATMEGA1284P-AU, Y6 8MHz LFXTAL083138

Commit message: Update project to KiCADv9.
Other:
- title: (none) -> DATALOGGER02A
