File: hw/sch_pcb/DATALOGGER02.kicad_pcb (KiCad board)
At the start: 4 copper layers, 101.1 x 60.5 mm, 160 parts, among them IC1 CY15B108QN-40SXI, IC2 FM3164-G, IC3 LTC4041EUFD#PBF, J1 HEADER_2x01_PARALLEL, J10 HEADER_2x05_PARALLEL, J11 HEADER_2x07_PARALLEL, J12 HEADER_2x05_PARALLEL, J13 HEADER_2x02_PARALLEL, J2 HEADER_2x01, J23 MCX, J24 HEADER_2x03_PARALLEL, J3 HEADER_2x03, J4 HEADER_2x03_PARALLEL, J5 HEADER_2x03_PARALLEL, J6 MCC-SD (kouka z modulu), J7 Conn_01x06_Female, J8 Conn_01x07_Female, J9 Conn_01x04_Female, Q1 DMP2045UQ-7, Q2 DMTH3002LPS, Q3 DMTH3002LPS, U1 ISL21080CIH320Z-TK, U10 TPS631000DRLR, U11 SX1262, U12 PE4259, U2 LM4041CIM3-1.2(neosazovat), U3 ATMEGA1284P-AU, U4 TXS0108EPW, U5 ICM-20948, U6 TPS22965-Q1, U7 MS5611-01BA, U8 MIC5504-1.8YM5-TR, U9 TPS631000DRLR, Y2 6pF crystal - 32.768kHz, Y3 32MHz, Y6 8MHz LFXTAL083138

Commit message: Desing improvements WIP.
Parts:
- added J14: Conn_01x06_Female, Connector_JST:JST_GH_SM06B-GHS-TB_1x06-1MP_P1.25mm_Horizontal, F.Cu at (130.4, 133.2)
- J3: footprint Mlab_Pin_Headers:Straight_2x03 -> Mlab_Pin_Headers:SMD_2x03_WO_paste
- moved C59 3.85 mm to (55.9, 89.5), turned to -90 degrees
- moved C51 1.30 mm to (73.0, 93.6)
Routing:
- net Net-(C59-Pad2): track 4.38 -> 2.22 mm
