File: hw/sch_pcb/DATALOGGER02.kicad_pcb (KiCad board)
At the start: 2 copper layers, 101.1 x 60.5 mm, 161 parts, among them IC1 CY15B108QN-40SXI, IC2 FM3164-G, IC3 LTC4041EUFD#PBF, J1 HEADER_2x01_PARALLEL, J10 HEADER_2x05_PARALLEL, J11 HEADER_2x07_PARALLEL, J12 HEADER_2x05_PARALLEL, J13 HEADER_2x02_PARALLEL, J14 Conn_01x06_Female, J2 HEADER_2x01, J23 VAL**, J24 HEADER_2x03_PARALLEL, J3 HEADER_2x03, J4 HEADER_2x03_PARALLEL, J5 HEADER_2x03_PARALLEL, J6 MCC-SD (kouka z modulu), J7 Conn_01x06_Female, J8 Conn_01x07_Female, J9 Conn_01x04_Female, Q1 DMP2045UQ-7, Q2 DMTH3002LPS, Q3 DMTH3002LPS, U1 ISL21080CIH320Z-TK, U10 TPS631000DRLR, U11 SX1262, U12 PE4259, U2 LM4041CIM3-1.2(neosazovat), U3 ATMEGA1284P-AU, U4 TXS0108EPW, U5 ICM-20948, U6 TPS22965-Q1, U7 MS5611-01BA, U8 MIC5504-1.8YM5-TR, U9 TPS631000DRLR, Y2 6pF crystal - 32.768kHz, Y3 32MHz, Y6 8MHz LFXTAL083138

Commit message: minor pcb layout fixes
Parts:
- moved R36 0.20 mm to (130.5, 101.9)
Routing:
- net +3.3V: track 381.7 -> 378.2 mm
- net MISO_SPI: track 93.6 -> 92.3 mm
- net +1V8: track 56.1 -> 54.9 mm
- net UNREG_POWER_INPUT: track 77.2 -> 76.1 mm
- net Net-(BT1-+): track 45.8 -> 44.7 mm
- net /Power_management/Vdc: track 124.3 -> 123.5 mm
- net Net-(U10-LX1): track 2.34 -> 1.63 mm
- net CS_FRAM: track 29.7 -> 29.0 mm
- net Net-(U10-LX2): track 2.40 -> 1.72 mm
- net /Peripherals/SCL_I2C_1V8: track 9.39 -> 8.71 mm
- net DIO_LORA: track 52.4 -> 53.1 mm
- net SCK_SPI: track 87.5 -> 86.9 mm
- net +5V: track 162.1 -> 161.5 mm
- net GND: track 179.4 -> 178.8 mm, vias 141 -> 140
- net PA0: track 34.0 -> 33.5 mm
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