File: hw/sch_pcb/Peripherals.kicad_sch (KiCad schematic)
At the start: 43 parts, among them IC1 CY15B108QN-40SXI, IC2 FM3164-G, J4 HEADER_2x03_PARALLEL, J6 MCC-SD (kouka z modulu), Q1 DMP2045UQ-7, U4 TXS0108EPW, U5 ICM-20948, U6 TPS22965-Q1, U7 MS5611-01BA, Y2 6pF crystal - 32.768kHz

Commit message: Update project to KiCADv9.
Other:
- title: (none) -> DATALOGGER02A
