File: hw/sch_pcb/Power_management.kicad_sch (KiCad schematic)
At the start: 46 parts, among them IC3 LTC4041EUFD#PBF, J24 HEADER_2x03_PARALLEL, J5 HEADER_2x03_PARALLEL, Q2 DMTH3002LPS, Q3 DMTH3002LPS, U10 TPS631000DRLR, U8 MIC5504-1.8YM5-TR, U9 TPS631000DRLR

Commit message: Update project to KiCADv9.
Other:
- title: (none) -> DATALOGGER02A
